File: BadgeThing.kicad_sch (KiCad schematic)
At the start: 56 parts, among them J1 USB_C_Receptacle_USB2.0, J2 Connector_Generic_Conn_01x02, SW1 BOOTSEL, SW2 ESP RESET, SW3 SW_Push, SW4 SW_Push, SW5 SW_Push, SW6 SW_Push, SW7 SW_Push, U2 W25Q32JVSS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

Commit message: Initial schematic
Parts:
- added D6: Greeen, LED_SMD:LED_0402_1005Metric_Pad0.77x0.64mm_HandSolder, symbol Device:LED_Small
- added J3: Ext 5V, Connector_PinHeader_2.54mm:PinHeader_1x02_P2.54mm_Vertical, symbol Connector_Generic:Conn_01x02
- added J4: SWD Header, Connector_PinHeader_2.54mm:PinHeader_1x03_P2.54mm_Vertical, symbol Connector_Generic:Conn_01x03
- added J5: ~, Connector_PinHeader_2.54mm:PinHeader_2x03_P2.54mm_Vertical, symbol Connector_Generic:Conn_02x03_Odd_Even
- added J6, J7: Conn_01x07, Connector_PinHeader_2.54mm:PinHeader_1x07_P2.54mm_Vertical, symbol Connector_Generic:Conn_01x07
- added J8: Conn_01x08, Connector_PinHeader_2.54mm:PinHeader_1x08_P2.54mm_Vertical, symbol Connector_Generic:Conn_01x08
- added R13, R14: 10K, Resistor_SMD:R_0402_1005Metric_Pad0.72x0.64mm_HandSolder, symbol Device:R_Small
- C1, C2, C3, C4, C5, C6: footprint (none) -> Capacitor_SMD:C_0402_1005Metric_Pad0.74x0.62mm_HandSolder
- J2: footprint (none) -> Connector_PinHeader_2.54mm:PinHeader_1x02_P2.54mm_Vertical
- JP1, JP2: footprint (none) -> Jumper:SolderJumper-2_P1.3mm_Open_RoundedPad1.0x1.5mm
- R1, R11, R12, R2: footprint (none) -> Resistor_SMD:R_0402_1005Metric_Pad0.72x0.64mm_HandSolder
- SW1: footprint Misc Footprints:TS-1187A-B-A-B -> Button_Switch_SMD:SW_Push_1P1T_NO_6x6mm_H9.5mm
- SW2: footprint (none) -> Button_Switch_SMD:SW_Push_1P1T_NO_6x6mm_H9.5mm
- SW3: value SW_Push -> Left; footprint (none) -> Button_Switch_SMD:SW_Push_1P1T_NO_6x6mm_H9.5mm
- SW4: value SW_Push -> Down; footprint (none) -> Button_Switch_SMD:SW_Push_1P1T_NO_6x6mm_H9.5mm
- SW5: value SW_Push -> Select; footprint (none) -> Button_Switch_SMD:SW_Push_1P1T_NO_6x6mm_H9.5mm
- SW6: value SW_Push -> Up; footprint (none) -> Button_Switch_SMD:SW_Push_1P1T_NO_6x6mm_H9.5mm
- SW7: value SW_Push -> Right; footprint (none) -> Button_Switch_SMD:SW_Push_1P1T_NO_6x6mm_H9.5mm
- U1: footprint (none) -> SSD1306 Pins:SSD1306 0.5mm Pitch
Connections:
- net +3V3: now also D6.2 (A), J5.2 (Pin_2), R13.1, R14.1
- net +5V: now also J3.2 (Pin_2)
- net BEEP: now also U3.8 (GPIO6); no longer U3.9 (GPIO7)
- net BTN1: now also U3.9 (GPIO7); no longer U3.11 (GPIO8)
- net BTN2: now also U3.11 (GPIO8); no longer U3.12 (GPIO9)
- net BTN3: now also U3.12 (GPIO9); no longer U3.13 (GPIO10)
- net BTN4: now also U3.13 (GPIO10); no longer U3.14 (GPIO11)
- net BTN5: now also U3.14 (GPIO11); no longer U3.15 (GPIO12)
- net GND: now also D6.1 (K), J3.1 (Pin_1), J4.2 (Pin_2), J5.4 (Pin_4)
- net MISO: no longer U5.10 (MISO)
- net MOSI: no longer U5.13 (MOSI)
- net SCLK: no longer U5.14 (SCLK)
- net SWCLK: now also J4.1 (Pin_1)
- net SWDIO: now also J4.3 (Pin_3)
- net WS2812B: now also U3.17 (GPIO14)
- net ESP_TX: now reaches U3.16 (GPIO13)
- net ESP_TX: now also U5.22 (GPIO1/TXD), J5.3 (Pin_3), R14.2
- net GP15: now reaches U3.18 (GPIO15)
- net GP15: now also J6.1 (Pin_1)
- net GP16: now reaches U3.27 (GPIO16)
- net GP16: now also J6.2 (Pin_2)
- net GP17: now reaches U3.28 (GPIO17)
- net GP17: now also J6.3 (Pin_3)
- net GP18: now reaches U3.29 (GPIO18)
- net GP18: now also J6.4 (Pin_4)
- net GP19: now reaches U3.30 (GPIO19)
- net GP19: now also J6.5 (Pin_5)
- net GP20: now reaches U3.31 (GPIO20)
- net GP20: now also J6.6 (Pin_6)
- net GP21: now reaches U3.32 (GPIO21)
- net GP21: now also J6.7 (Pin_7)
- net GP22: now reaches U3.34 (GPIO22)
- net GP22: now also J7.1 (Pin_1)
- net GP23: now reaches U3.35 (GPIO23)
- net GP23: now also J7.2 (Pin_2)
- net GP24: now reaches U3.36 (GPIO24)
- net GP24: now also J7.3 (Pin_3)
- net GP26: now reaches U3.38 (GPIO26_ADC0)
- net GP26: now also J7.4 (Pin_4)
- net GP27: now reaches U3.39 (GPIO27_ADC1)
- net GP27: now also J7.5 (Pin_5)
- net GP28: now reaches U3.40 (GPIO28_ADC2)
- net GP28: now also J7.6 (Pin_6)
- net GP29: now reaches U3.41 (GPIO29_ADC3)
- net GP29: now also J7.7 (Pin_7)
- net ESP15: now reaches U5.16 (GPIO15)
- net ESP15: now also J8.7 (Pin_7)
- net ESP2: now reaches U5.17 (GPIO2)
- net ESP2: now also J8.1 (Pin_1)
- net ESP0: now reaches U5.18 (GPIO0)
- net ESP0: now also J5.6 (Pin_6)
- net ESP4: now reaches U5.19 (GPIO4)
- net ESP4: now also J8.2 (Pin_2)
- net ESP5: now reaches U5.20 (GPIO5)
- net ESP5: now also J8.3 (Pin_3)
- net ESP_RX: now reaches U5.21 (GPIO3/RXD)
- net ESP_RX: now also U3.15 (GPIO12), J5.5 (Pin_5), R13.2
- net ESP_EN: now reaches U5.3 (EN)
- net ESP_EN: now also J5.1 (Pin_1)
- net ESP16: now reaches U5.4 (GPIO16)
- net ESP16: now also J8.8 (Pin_8)
- net ESP14: now reaches U5.5 (GPIO14)
- net ESP14: now also J8.6 (Pin_6)
- net ESP12: now reaches U5.6 (GPIO12)
- net ESP12: now also J8.4 (Pin_4)
- net ESP13: now reaches U5.7 (GPIO13)
- net ESP13: now also J8.5 (Pin_5)
- net CS2: no longer names the net of U5.9 (CS0)
- net CS2: no longer U3.8 (GPIO6)
- no-connect marks 10 -> 16
Other:
- note added: "Do Not Use to keep compatibility with ESP-12S"
- note added: "ESP GPIO"
- note added: "GPIO Header 1"
- note added: "GPIO Header 2"
- note added: "ICSP"
- note added: "Power LED"
- note added: "Progam Flash"
- note added: "SWD"
- note removed: "Flash Memory"
- moved on the sheet: C10, C16, C19, C20, C21, D1, R10, R7, SW2, SW3, SW5, SW6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

Commit message: RP2040/OLED circuits, basic component placement
Parts:
- J4: footprint Connector_PinHeader_2.54mm:PinHeader_1x03_P2.54mm_Vertical -> Connector_PinHeader_1.27mm:PinHeader_1x03_P1.27mm_Vertical
Other:
- note added: "ABLS-12.000MHZ-B4-T"
- note removed: "12MHz Crystal"
Changed lines of the file:
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@@
     (effects (font (size 1.27 1.27)) (justify left bottom))
   )
-  (text "12MHz Crystal" (at 203.835 41.275 0)
-    (effects (font (size 1.27 1.27)) (justify left bottom))
+  (text "ABLS-12.000MHZ-B4-T" (at 203.2 41.275 0)
+    (effects (font (size 1 1)) (justify left bottom))
   )
   (text "ICSP" (at 67.183 136.779 0)
@@
       (effects (font (size 1.27 1.27)) (justify left))
     )
-    (property "Footprint" "Connector_PinHeader_2.54mm:PinHeader_1x03_P2.54mm_Vertical" (at 234.95 107.315 0)
-      (effects (font (size 1.27 1.27)) hide)
-    )
+    (property "Footprint" "Connector_PinHeader_1.27mm:PinHeader_1x03_P1.27mm_Vertical" (at 234.95 107.315 0)
+      (effects (font (size 1.27 1.27)) hide)
+    )
